File: hp34401a_oled.sch (KiCad schematic (older format))
At the start: 32 parts, among them J1 USB_B_Micro, J2 DISPLAY, J3 UART, J4 FP, J5 DISPLAYPWR, U1 STM32F103C8Tx, U2 LM1117-3.3, Y1 8M

Commit message: Tweak size, footprints, generate gerber
Parts:
- added C7: 0.1uF, Capacitor_SMD:C_0603_1608Metric, symbol Device:C
- added U3: AT24C02, Package_SO:SOIC-8_3.9x4.9mm_P1.27mm, symbol Memory_EEPROM:AT24CS02-SSHM
- J1: footprint Connector_USB:USB_Micro-B_Wuerth_614105150721_Vertical_CircularHoles -> Connector_USB:USB_Micro-B_Wuerth_614105150721_Vertical
Connections:
- net labels added: SCL, SDA
- wire segments 149 -> 168
- no-connect marks 16 -> 14
Other:
- moved on the sheet: U2
